File: Schematics/Euclidean_Rhythms/Eudlidean_Rhythms.kicad_pcb (KiCad board)
At the start: 2 copper layers, 87.6 x 56.5 mm, 67 parts, among them J1 POWER, J2 INPUTS, J3 LEDS, J4 PROB, J5 OUTPUTS, J6 OLED, U1 TL074, U2 TL074

Commit message: Add files via upload
Parts:
- removed the D3 at (93.4, 101.0)
- J2: footprint Connector_PinHeader_2.54mm:PinHeader_1x08_P2.54mm_Vertical -> Connector_PinHeader_2.54mm:PinHeader_1x09_P2.54mm_Vertical
- moved C8 43.1 mm to (138.4, 81.9), turned to -90 degrees
- moved A1 40.0 mm to (122.0, 103.6)
- moved R16 40.0 mm to (161.9, 129.5)
- moved C6 40.0 mm to (164.4, 95.2)
- moved C7 40.0 mm to (164.4, 119.4)
- moved R13 40.0 mm to (148.0, 106.6)
- moved R17 40.0 mm to (161.9, 109.2)
- moved R33 40.0 mm to (161.9, 105.4)
- moved R6 40.0 mm to (148.0, 90.1)
- moved C2 40.0 mm to (132.7, 118.6)
- moved C3 40.0 mm to (156.8, 127.0)
- moved C4 40.0 mm to (178.4, 95.2)
- moved D3 40.0 mm to (128.3, 87.0)
- moved D6 40.0 mm to (179.1, 109.2)
- moved D7 40.0 mm to (179.1, 124.5)
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Connections:
- A1 pad 7: ESW -> E2
- A1 pad 8: E2 -> ESW
- J2 pad 3: E2 -> ESW
- J2 pad 4: ESW -> E2
Routing:
- net TRG: track 24.0 -> 20.8 mm
- net +5V: track 84.4 -> 81.4 mm
- net Net-(D3-A): track 5.07 -> 2.49 mm
- net Net-(D1-A): track 13.7 -> 11.2 mm
- net GND: track 71.1 -> 71.9 mm
- net Net-(A1-A6): track 75.4 -> 76.1 mm
Other:
- board text added: "EUCLIDEAN RHYTHMS or 6-CHANNEL SEQUENCER"
- board text added: "INSPIRED BY THE ORIGINAL HAGIWO DESIGNS"
- board text removed: "EUCLIDEAN RHYTHMS"
- board text removed: "INSPIRED BY THE ORIGINAL HAGIWO DESIGN"
