File: Schematics/Euclidean_Rhythms/Eudlidean_Rhythms.kicad_sch (KiCad schematic)
At the start: 74 parts, among them J1 POWER, J10 OUT1, J2 INPUTS, J3 LEDS, J4 PROB, J5 OUTPUTS, J6 OLED, J7 CLK, J8 PROB, J9 ZERO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

Commit message: Add files via upload
Parts:
- J2: footprint Connector_PinHeader_2.54mm:PinHeader_1x08_P2.54mm_Vertical -> Connector_PinHeader_2.54mm:PinHeader_1x09_P2.54mm_Vertical
Connections:
- net E2: now also A1.7 (D4), J2.4 (Pin_4); no longer A1.8 (D5), J2.3 (Pin_3)
- net ESW: now also A1.8 (D5), J2.3 (Pin_3); no longer A1.7 (D4), J2.4 (Pin_4)
Other:
- note added: "R8, R10, R13, R15, R28 & R30 10k for red LED, 39k for green"
- moved on the sheet: D9, J10, J7, J8, J9, RV1, RV2, SW1, SW2, SW3, Z1
